Commit message: Add files via upload

File: my_mobile_robot/urdf/robot.urdf (robot description, URDF)
Before this commit: robot robot, 5 links, 4 joints
Links:
- added link Jetson; visual mesh filename=package://my_mobile_robot/STL/Jetson.STL scale=0.001 0.001 0.001
Joints:
- added joint Jetson_joint: type fixed, parent chassis, child Jetson, origin xyz=0 0 0.145 rpy=0 0 0
- joint caster_wheel_joint: axis 0 1 0 -> (none); origin xyz=-0.11 0.06 -0.015 rpy=1.56 0 0 -> xyz=0 0 0 rpy=0 0 0; type continuous -> fixed
- joint chassis_joint: origin xyz=0 0 0 -> xyz=0 0 0 rpy=0 0 0
- joint left_wheel: axis 0 0 1 -> (none); origin xyz=0.102 0.02 0.030 rpy=1.56 0 0 -> xyz=0.005 0.085 0.030 rpy=0 0 1.57
- joint right_wheel: axis 0 0 -1 -> (none); origin xyz=-0.105 0.02 0.030 rpy=1.56 0 0 -> xyz=0 -0.105 0.030 rpy=0 0 -1.57
