Commit message: Add files via upload

File: my_mobile_robot/urdf/robot_core.xacro (robot description, xacro)
@@ -44,4 +44,28 @@
         </xacro:inertial_box>
     </link>
+    <!-- Jetson -->
+    <joint name="Jetson_joint" type="fixed">
+        <parent link="base_link" />
+        <child link="Jetson" />
+        <origin xyz="0 0 0" rpy="0 0 0"/>
+    </joint>
+    <link name="Jetson">
+        <visual>
+            <geometry>
+              <mesh filename="package://my_mobile_robot/STL/Jetson.STL" scale="0.001 0.001 0.001"/>
+            </geometry>
+            <origin xyz="-0.06 0.05 0.122" rpy="0 0 -1.57"/>
+            <material name="blue"/>
+        </visual>
+        <!--<collision>
+            <origin xyz="0.15 0 0.075" />
+            <geometry>
+                <box size="0.3 0.3 0.15" />
+            </geometry>
+        </collision> -->
+        <xacro:inertial_box mass="0.5" x="0.3" y="0.3" z="0.15">
+            <origin xyz="-0.11 0.05 -0.015" rpy="1.56 0 0"/>
+        </xacro:inertial_box>
+    </link>
     <!-- LEFT WHEEL LINK -->
     <joint name="left_wheel" type="continuous">
@@ -57,5 +81,5 @@
             </geometry>
             <origin xyz="-0.22 -0.045 -0.04" rpy="0 0 0"/>
-            <material name="white"/>
+            <material name="orange"/>
         </visual>
         <!--<collision>
@@ -90,5 +114,5 @@
             </geometry>
             <origin xyz="0 -0.045 -0.04" rpy="0 0 0"/>
-            <material name="white"/>
+            <material name="orange"/>
         </visual>
         <!--<collision>
@@ -150,5 +174,5 @@
               <mesh filename="package://my_mobile_robot/STL/FreeBall.STL" scale="0.001 0.001 0.001"/>
             </geometry>
-            <origin xyz="-0.11 0.06 -0.015" rpy="1.56 0 0"/>
+            <origin xyz="-0.125 0.15 -0.015" rpy="1.56 0 0"/>
             <material name="white"/>
         </visual>
@@ -169,5 +193,5 @@
                 <cylinder radius="0.02" length="0.02" /> <!-- Example shape, adjust as needed -->
             </geometry>
-            <material name="blue" /> <!-- Example material, adjust as needed -->
+            <material name="black" /> <!-- Example material, adjust as needed -->
         </visual>
         <!--<collision>
@@ -183,5 +207,5 @@
         <parent link="chassis"/>
         <child link="lidar_link"/>
-        <origin xyz="0 0 0.13" rpy="0 0 0"/>
+        <origin xyz="-0.015 -0.012 0.198" rpy="0 0 0"/>
     </joint>
     <gazebo reference="lidar_link">

Commit message: Add files via upload

File: my_mobile_robot/urdf/robot_core.xacro (robot description, xacro)
@@ -24,5 +24,5 @@
         <parent link="base_link" />
         <child link="chassis" />
-        <origin xyz="0 0 0" rpy="0 0 0"/>
+        <origin xyz="0 0 0" rpy="0 0 -1.57"/>
     </joint>
     <link name="chassis">
@@ -31,5 +31,5 @@
               <mesh filename="package://my_mobile_robot/STL/Chassis.STL" scale="0.001 0.001 0.001"/>
             </geometry>
-            <origin xyz="-0.11 0.05 -0.015" rpy="1.56 0 0"/>
+            <origin xyz="-0.05 -0.1 -0.016" rpy="1.57 0 1.57"/>
             <material name="white"/>
         </visual>
@@ -41,12 +41,12 @@
         </collision> -->
         <xacro:inertial_box mass="0.5" x="0.3" y="0.3" z="0.15">
-            <origin xyz="-0.11 0.05 -0.015" rpy="1.56 0 0"/>
+            <origin xyz="0 0 0" rpy="1.57 0 1.57"/>
         </xacro:inertial_box>
     </link>
     <!-- Jetson -->
     <joint name="Jetson_joint" type="fixed">
-        <parent link="base_link" />
+        <parent link="chassis" />
         <child link="Jetson" />
-        <origin xyz="0 0 0" rpy="0 0 0"/>
+        <origin xyz="0 0 0.145" rpy="0 0 0"/>
     </joint>
     <link name="Jetson">
@@ -55,5 +55,5 @@
               <mesh filename="package://my_mobile_robot/STL/Jetson.STL" scale="0.001 0.001 0.001"/>
             </geometry>
-            <origin xyz="-0.06 0.05 0.122" rpy="0 0 -1.57"/>
+            <origin xyz="-0.035 -0.045 -0.025" rpy="0 0 0"/>
             <material name="blue"/>
         </visual>
@@ -65,5 +65,5 @@
         </collision> -->
         <xacro:inertial_box mass="0.5" x="0.3" y="0.3" z="0.15">
-            <origin xyz="-0.11 0.05 -0.015" rpy="1.56 0 0"/>
+            <origin xyz="-0.06 0.05 0.122" rpy="0 0 0"/>
         </xacro:inertial_box>
     </link>
@@ -72,5 +72,5 @@
         <parent link="base_link" />
         <child link="left_wheel_link" />
-        <origin xyz="0.102 0.02 0.030" rpy="1.56 0 0"/>
+        <origin xyz="0.102 -0.005 0.030" rpy="0 0 -1.57"/>
         <dynamics damping="0.5" friction="100.0" />
     </joint>
@@ -80,5 +80,5 @@
               <mesh filename="package://my_mobile_robot/STL/wheels_step-1.STL" scale="0.001 0.001 0.001"/>
             </geometry>
-            <origin xyz="-0.22 -0.045 -0.04" rpy="0 0 0"/>
+            <origin xyz="0.055 -0.22 -0.04" rpy="0 0 1.57"/>
             <material name="orange"/>
         </visual>
@@ -89,5 +89,5 @@
         </collision>-->
         <xacro:inertial_cylinder mass="0.1" length="0.04" radius="0.05">
-            <origin xyz="0 0 0" rpy="0 0 0" />
+            <origin xyz="0.075 -0.22 -0.02" rpy="0 0 1.57" />
         </xacro:inertial_cylinder>
     </link>
@@ -105,5 +105,5 @@
         <parent link="base_link" />
         <child link="right_wheel_link" />
-        <origin xyz="-0.105 0.02 0.030" rpy="1.56 0 0"/>
+        <origin xyz="-0.105 -0.005 0.030" rpy="0 0 -1.57"/>
         <dynamics damping="0.5" friction="100.0" />
     </joint>
@@ -113,5 +113,5 @@
               <mesh filename="package://my_mobile_robot/STL/wheels_step-2.STL" scale="0.001 0.001 0.001"/>
             </geometry>
-            <origin xyz="0 -0.045 -0.04" rpy="0 0 0"/>
+            <origin xyz="0.055 -0.005 -0.04" rpy="0 0 1.57"/>
             <material name="orange"/>
         </visual>
@@ -122,5 +122,5 @@
         </collision>-->
         <xacro:inertial_cylinder mass="0.1" length="0.04" radius="0.05">
-            <origin xyz="0 0 0" rpy="0 0 0" />
+            <origin xyz="0.075 -0.005 0" rpy="0 0 1.57" />
         </xacro:inertial_cylinder>
     </link>
@@ -174,5 +174,5 @@
               <mesh filename="package://my_mobile_robot/STL/FreeBall.STL" scale="0.001 0.001 0.001"/>
             </geometry>
-            <origin xyz="-0.125 0.15 -0.015" rpy="1.56 0 0"/>
+            <origin xyz="-0.15 -0.115 -0.015" rpy="1.57 0 1.57"/>
             <material name="white"/>
         </visual>
@@ -183,5 +183,5 @@
         </collision>-->
         <xacro:inertial_sphere mass="0.1" radius="0.05">
-            <origin xyz="0 0 0" rpy="0 0 0" />
+            <origin xyz="0.125 0.15 -0.015" rpy="1.57 0 1.57" />
         </xacro:inertial_sphere>
     </link>
@@ -207,5 +207,5 @@
         <parent link="chassis"/>
         <child link="lidar_link"/>
-        <origin xyz="-0.015 -0.012 0.198" rpy="0 0 0"/>
+        <origin xyz="0.0105 -0.005 0.199" rpy="0 0 0"/>
     </joint>
     <gazebo reference="lidar_link">

Commit message: Lastest update

File: my_mobile_robot/urdf/robot_core.xacro (robot description, xacro)
@@ -24,5 +24,5 @@
         <parent link="base_link" />
         <child link="chassis" />
-        <origin xyz="0 0 0" rpy="0 0 0"/>
+        <origin xyz="0 0 0" rpy="0 0 -1.57"/>
     </joint>
     <link name="chassis">
@@ -31,5 +31,5 @@
               <mesh filename="package://my_mobile_robot/STL/Chassis.STL" scale="0.001 0.001 0.001"/>
             </geometry>
-            <origin xyz="-0.11 0.05 -0.015" rpy="1.56 0 0"/>
+            <origin xyz="-0.05 -0.1 -0.016" rpy="1.57 0 1.57"/>
             <material name="white"/>
         </visual>
@@ -41,5 +41,29 @@
         </collision> -->
         <xacro:inertial_box mass="0.5" x="0.3" y="0.3" z="0.15">
-            <origin xyz="-0.11 0.05 -0.015" rpy="1.56 0 0"/>
+            <origin xyz="0 0 0" rpy="1.57 0 1.57"/>
+        </xacro:inertial_box>
+    </link>
+    <!-- Jetson -->
+    <joint name="Jetson_joint" type="fixed">
+        <parent link="chassis" />
+        <child link="Jetson" />
+        <origin xyz="0 0 0.145" rpy="0 0 0"/>
+    </joint>
+    <link name="Jetson">
+        <visual>
+            <geometry>
+              <mesh filename="package://my_mobile_robot/STL/Jetson.STL" scale="0.001 0.001 0.001"/>
+            </geometry>
+            <origin xyz="-0.035 -0.045 -0.025" rpy="0 0 0"/>
+            <material name="blue"/>
+        </visual>
+        <!--<collision>
+            <origin xyz="0.15 0 0.075" />
+            <geometry>
+                <box size="0.3 0.3 0.15" />
+            </geometry>
+        </collision> -->
+        <xacro:inertial_box mass="0.5" x="0.3" y="0.3" z="0.15">
+            <origin xyz="-0.06 0.05 0.122" rpy="0 0 0"/>
         </xacro:inertial_box>
     </link>
@@ -48,5 +72,5 @@
         <parent link="base_link" />
         <child link="left_wheel_link" />
-        <origin xyz="0.102 0.02 0.030" rpy="1.56 0 0"/>
+        <origin xyz="0.102 -0.005 0.030" rpy="0 0 -1.57"/>
         <dynamics damping="0.5" friction="100.0" />
     </joint>
@@ -56,6 +80,6 @@
               <mesh filename="package://my_mobile_robot/STL/wheels_step-1.STL" scale="0.001 0.001 0.001"/>
             </geometry>
-            <origin xyz="-0.22 -0.045 -0.04" rpy="0 0 0"/>
-            <material name="white"/>
+            <origin xyz="0.055 -0.22 -0.04" rpy="0 0 1.57"/>
+            <material name="orange"/>
         </visual>
         <!--<collision>
@@ -65,5 +89,5 @@
         </collision>-->
         <xacro:inertial_cylinder mass="0.1" length="0.04" radius="0.05">
-            <origin xyz="0 0 0" rpy="0 0 0" />
+            <origin xyz="0.075 -0.22 -0.02" rpy="0 0 1.57" />
         </xacro:inertial_cylinder>
     </link>
@@ -81,5 +105,5 @@
         <parent link="base_link" />
         <child link="right_wheel_link" />
-        <origin xyz="-0.105 0.02 0.030" rpy="1.56 0 0"/>
+        <origin xyz="-0.105 -0.005 0.030" rpy="0 0 -1.57"/>
         <dynamics damping="0.5" friction="100.0" />
     </joint>
@@ -89,6 +113,6 @@
               <mesh filename="package://my_mobile_robot/STL/wheels_step-2.STL" scale="0.001 0.001 0.001"/>
             </geometry>
-            <origin xyz="0 -0.045 -0.04" rpy="0 0 0"/>
-            <material name="white"/>
+            <origin xyz="0.055 -0.005 -0.04" rpy="0 0 1.57"/>
+            <material name="orange"/>
         </visual>
         <!--<collision>
@@ -98,5 +122,5 @@
         </collision>-->
         <xacro:inertial_cylinder mass="0.1" length="0.04" radius="0.05">
-            <origin xyz="0 0 0" rpy="0 0 0" />
+            <origin xyz="0.075 -0.005 0" rpy="0 0 1.57" />
         </xacro:inertial_cylinder>
     </link>
@@ -150,5 +174,5 @@
               <mesh filename="package://my_mobile_robot/STL/FreeBall.STL" scale="0.001 0.001 0.001"/>
             </geometry>
-            <origin xyz="-0.11 0.06 -0.015" rpy="1.56 0 0"/>
+            <origin xyz="-0.15 -0.115 -0.015" rpy="1.57 0 1.57"/>
             <material name="white"/>
         </visual>
@@ -159,5 +183,5 @@
         </collision>-->
         <xacro:inertial_sphere mass="0.1" radius="0.05">
-            <origin xyz="0 0 0" rpy="0 0 0" />
+            <origin xyz="0.125 0.15 -0.015" rpy="1.57 0 1.57" />
         </xacro:inertial_sphere>
     </link>
@@ -169,5 +193,5 @@
                 <cylinder radius="0.02" length="0.02" /> <!-- Example shape, adjust as needed -->
             </geometry>
-            <material name="blue" /> <!-- Example material, adjust as needed -->
+            <material name="black" /> <!-- Example material, adjust as needed -->
         </visual>
         <!--<collision>
@@ -183,5 +207,5 @@
         <parent link="chassis"/>
         <child link="lidar_link"/>
-        <origin xyz="0 0 0.13" rpy="0 0 0"/>
+        <origin xyz="0.0105 -0.005 0.199" rpy="0 0 0"/>
     </joint>
     <gazebo reference="lidar_link">

Commit message: Add files via upload

File: my_mobile_robot/urdf/robot_core.xacro (robot description, xacro)
@@ -24,5 +24,5 @@
         <parent link="base_link" />
         <child link="chassis" />
-        <origin xyz="0 0 0" rpy="0 0 -1.57"/>
+        <origin xyz="0 0 0" rpy="0 0 0"/>
     </joint>
     <link name="chassis">
@@ -72,5 +72,5 @@
         <parent link="base_link" />
         <child link="left_wheel_link" />
-        <origin xyz="0.102 -0.005 0.030" rpy="0 0 -1.57"/>
+        <origin xyz="0.005 0.085 0.030" rpy="0 0 1.57"/>
         <dynamics damping="0.5" friction="100.0" />
     </joint>
@@ -80,5 +80,5 @@
               <mesh filename="package://my_mobile_robot/STL/wheels_step-1.STL" scale="0.001 0.001 0.001"/>
             </geometry>
-            <origin xyz="0.055 -0.22 -0.04" rpy="0 0 1.57"/>
+            <origin xyz="-0.198 -0.055 -0.04" rpy="0 0 0"/>
             <material name="orange"/>
         </visual>
@@ -89,5 +89,5 @@
         </collision>-->
         <xacro:inertial_cylinder mass="0.1" length="0.04" radius="0.05">
-            <origin xyz="0.075 -0.22 -0.02" rpy="0 0 1.57" />
+            <origin xyz="0.075 -0.22 -0.02" rpy="0 0 0" />
         </xacro:inertial_cylinder>
     </link>
@@ -105,5 +105,5 @@
         <parent link="base_link" />
         <child link="right_wheel_link" />
-        <origin xyz="-0.105 -0.005 0.030" rpy="0 0 -1.57"/>
+        <origin xyz="0 -0.105 0.030" rpy="0 0 -1.57"/>
         <dynamics damping="0.5" friction="100.0" />
     </joint>
@@ -113,5 +113,5 @@
               <mesh filename="package://my_mobile_robot/STL/wheels_step-2.STL" scale="0.001 0.001 0.001"/>
             </geometry>
-            <origin xyz="0.055 -0.005 -0.04" rpy="0 0 1.57"/>
+            <origin xyz="-0.0205 -0.04 -0.04" rpy="0 0 0"/>
             <material name="orange"/>
         </visual>

Commit message: for create Video nah

File: my_mobile_robot/urdf/robot_core.xacro (robot description, xacro)
@@ -24,5 +24,5 @@
         <parent link="base_link" />
         <child link="chassis" />
-        <origin xyz="0 0 0" rpy="0 0 -1.57"/>
+        <origin xyz="0 0 0" rpy="0 0 0"/>
     </joint>
     <link name="chassis">
@@ -72,5 +72,5 @@
         <parent link="base_link" />
         <child link="left_wheel_link" />
-        <origin xyz="0.102 -0.005 0.030" rpy="0 0 -1.57"/>
+        <origin xyz="0.005 0.085 0.030" rpy="0 0 1.57"/>
         <dynamics damping="0.5" friction="100.0" />
     </joint>
@@ -80,5 +80,5 @@
               <mesh filename="package://my_mobile_robot/STL/wheels_step-1.STL" scale="0.001 0.001 0.001"/>
             </geometry>
-            <origin xyz="0.055 -0.22 -0.04" rpy="0 0 1.57"/>
+            <origin xyz="-0.198 -0.055 -0.04" rpy="0 0 0"/>
             <material name="orange"/>
         </visual>
@@ -89,5 +89,5 @@
         </collision>-->
         <xacro:inertial_cylinder mass="0.1" length="0.04" radius="0.05">
-            <origin xyz="0.075 -0.22 -0.02" rpy="0 0 1.57" />
+            <origin xyz="0.075 -0.22 -0.02" rpy="0 0 0" />
         </xacro:inertial_cylinder>
     </link>
@@ -105,5 +105,5 @@
         <parent link="base_link" />
         <child link="right_wheel_link" />
-        <origin xyz="-0.105 -0.005 0.030" rpy="0 0 -1.57"/>
+        <origin xyz="0 -0.105 0.030" rpy="0 0 -1.57"/>
         <dynamics damping="0.5" friction="100.0" />
     </joint>
@@ -113,5 +113,5 @@
               <mesh filename="package://my_mobile_robot/STL/wheels_step-2.STL" scale="0.001 0.001 0.001"/>
             </geometry>
-            <origin xyz="0.055 -0.005 -0.04" rpy="0 0 1.57"/>
+            <origin xyz="-0.0205 -0.04 -0.04" rpy="0 0 0"/>
             <material name="orange"/>
         </visual>
@@ -224,5 +224,5 @@
                 </scan>
                 <range>
-                    <min>0.3</min>
+                    <min>0.15</min>
                     <max>12</max>
                 </range>

Commit message: Finished

File: my_mobile_robot/urdf/robot_core.xacro (robot description, xacro)
@@ -29,15 +29,15 @@
         <visual>
             <geometry>
-              <mesh filename="package://my_mobile_robot/STL/Chassis.STL" scale="0.001 0.001 0.001"/>
+                <mesh filename="package://my_mobile_robot/STL/Chassis.STL" scale="0.001 0.001 0.001"/>
             </geometry>
             <origin xyz="-0.05 -0.1 -0.016" rpy="1.57 0 1.57"/>
             <material name="white"/>
         </visual>
-        <!--<collision>
-            <origin xyz="0.15 0 0.075" />
-            <geometry>
-                <box size="0.3 0.3 0.15" />
-            </geometry>
-        </collision> -->
+        <collision>
+            <geometry>
+                <mesh filename="package://my_mobile_robot/STL/Chassis.STL" scale="0.001 0.001 0.001"/>
+            </geometry>
+            <origin xyz="-0.05 -0.1 -0.016" rpy="1.57 0 1.57"/>
+        </collision>
         <xacro:inertial_box mass="0.5" x="0.3" y="0.3" z="0.15">
             <origin xyz="0 0 0" rpy="1.57 0 1.57"/>
@@ -49,4 +49,5 @@
         <child link="Jetson" />
         <origin xyz="0 0 0.145" rpy="0 0 0"/>
+        <dynamics damping="0.5" friction="100.0" />
     </joint>
     <link name="Jetson">
@@ -58,12 +59,12 @@
             <material name="blue"/>
         </visual>
-        <!--<collision>
-            <origin xyz="0.15 0 0.075" />
-            <geometry>
-                <box size="0.3 0.3 0.15" />
-            </geometry>
-        </collision> -->
-        <xacro:inertial_box mass="0.5" x="0.3" y="0.3" z="0.15">
-            <origin xyz="-0.06 0.05 0.122" rpy="0 0 0"/>
+        <collision>
+            <geometry>
+             <mesh filename="package://my_mobile_robot/STL/Jetson.STL" scale="0.001 0.001 0.001"/>
+            </geometry>
+            <origin xyz="-0.035 -0.045 -0.025" rpy="0 0 0"/>
+        </collision>
+        <xacro:inertial_box mass="0" x="0.3" y="0.3" z="0.15">
+            <origin xyz="0 0 0" rpy="0 0 0"/>
         </xacro:inertial_box>
     </link>
@@ -72,5 +73,6 @@
         <parent link="base_link" />
         <child link="left_wheel_link" />
-        <origin xyz="0.005 0.085 0.030" rpy="0 0 1.57"/>
+        <origin xyz="0.007 0.085 0.034" rpy="-1.57 0 0"/>
+        <axis xyz="0 0 1" />
         <dynamics damping="0.5" friction="100.0" />
     </joint>
@@ -80,14 +82,15 @@
               <mesh filename="package://my_mobile_robot/STL/wheels_step-1.STL" scale="0.001 0.001 0.001"/>
             </geometry>
-            <origin xyz="-0.198 -0.055 -0.04" rpy="0 0 0"/>
+            <origin xyz="0.0455 -0.0495 -0.2" rpy="0 -1.57 0"/>
             <material name="orange"/>
         </visual>
-        <!--<collision>
-            <geometry>
-                <cylinder radius="0.05" length="0.04" />
-            </geometry>
-        </collision>-->
+        <collision>
+            <geometry>
+                <mesh filename="package://my_mobile_robot/STL/wheels_step-1.STL" scale="0.001 0.001 0.001"/>
+            </geometry>
+            <origin xyz="0.0455 -0.0495 -0.2" rpy="0 -1.57 0"/>
+        </collision>
         <xacro:inertial_cylinder mass="0.1" length="0.04" radius="0.05">
-            <origin xyz="0.075 -0.22 -0.02" rpy="0 0 0" />
+            <origin xyz="0 0 0" rpy="0 0 0"/>
         </xacro:inertial_cylinder>
     </link>
@@ -105,5 +108,6 @@
         <parent link="base_link" />
         <child link="right_wheel_link" />
-        <origin xyz="0 -0.105 0.030" rpy="0 0 -1.57"/>
+        <origin xyz="0.008 -0.105 0.033" rpy="1.57 0 0"/>
+        <axis xyz="0 0 -1" />
         <dynamics damping="0.5" friction="100.0" />
     </joint>
@@ -113,14 +117,15 @@
               <mesh filename="package://my_mobile_robot/STL/wheels_step-2.STL" scale="0.001 0.001 0.001"/>
             </geometry>
-            <origin xyz="-0.0205 -0.04 -0.04" rpy="0 0 0"/>
+            <origin xyz="-0.0455 -0.0495 0.007" rpy="0 1.57 0"/>
             <material name="orange"/>
         </visual>
-        <!--<collision>
-            <geometry>
-                <cylinder radius="0.05" length="0.04" />
-            </geometry>
-        </collision>-->
+        <collision>
+            <geometry>
+                <mesh filename="package://my_mobile_robot/STL/wheels_step-2.STL" scale="0.001 0.001 0.001"/>
+              </geometry>
+              <origin xyz="-0.0455 -0.0495 0.007" rpy="0 1.57 0"/>
+        </collision>
         <xacro:inertial_cylinder mass="0.1" length="0.04" radius="0.05">
-            <origin xyz="0.075 -0.005 0" rpy="0 0 1.57" />
+            <origin xyz="0 0 0" rpy="0 0 0"/>
         </xacro:inertial_cylinder>
     </link>
@@ -177,11 +182,12 @@
             <material name="white"/>
         </visual>
-        <!--<collision>
-            <geometry>
-                <sphere radius="0.05" />
-            </geometry>
-        </collision>-->
+        <collision>
+            <geometry>
+                <mesh filename="package://my_mobile_robot/STL/FreeBall.STL" scale="0.001 0.001 0.001"/>
+            </geometry>
+            <origin xyz="-0.15 -0.115 -0.015" rpy="1.57 0 1.57"/>
+        </collision>
         <xacro:inertial_sphere mass="0.1" radius="0.05">
-            <origin xyz="0.125 0.15 -0.015" rpy="1.57 0 1.57" />
+            <origin xyz="0 0 0" rpy="1.57 0 1.57"/>
         </xacro:inertial_sphere>
     </link>
@@ -195,10 +201,10 @@
             <material name="black" /> <!-- Example material, adjust as needed -->
         </visual>
-        <!--<collision>
-            Collision properties of the lidar sensor
+        <collision>
+            <!--Collision properties of the lidar sensor-->
             <geometry>
                 <cylinder radius="0.03" length="0.06" />
             </geometry>
-        </collision> -->
+        </collision>
         <!-- Define inertial properties if necessary -->
     </link>
